Commit message: urdf for virtual robot

File: iter_moveit/m1n6s_robotiq85_moveit_config/urdf/m1n6s.xacro (robot description, xacro)
@@ -1,4 +1,4 @@
 <?xml version="1.0"?>
-<!-- m1_4n refers to mico v1 6DOF non-spherical -->
+<!-- m1_6n refers to mico v1 6DOF non-spherical -->
 <root xmlns:xi="http://www.w3.org/2001/XInclude"
     xmlns:gazebo="http://playerstage.sourceforge.net/gazebo/xmlschema/#gz"
@@ -15,5 +15,4 @@
     xmlns:xacro="http://ros.org/wiki/xacro">
     <xacro:include filename="$(find kinova_description)/urdf/kinova_common.xacro" />
-    <xacro:include filename="$(find kinova_description)/urdf/kinova_finger_set.xacro" />
     <!-- Import all Gazebo-customization elements -->
     <xacro:include filename="$(find kinova_description)/urdf/kinova.gazebo" />
@@ -22,5 +21,7 @@
     <xacro:property name="link_2_mesh" value="arm_mico" />
     <xacro:property name="link_3_mesh" value="forearm_mico" />
-    <xacro:property name="link_4_mesh" value="hand_2finger" />
+    <xacro:property name="link_4_mesh" value="wrist" />
+    <xacro:property name="link_5_mesh" value="wrist" />
+    <xacro:property name="link_6_mesh" value="hand_2finger" />
     <!--Used for conditional arguments for setting inertial parameters
         base 0, shoulder 1, arm 2, forearm 3, wrist 4, arm_mico 5,
@@ -33,5 +34,7 @@
     <xacro:property name="link_2_mesh_no" value="5" />
     <xacro:property name="link_3_mesh_no" value="10" />
-    <xacro:property name="link_4_mesh_no" value="56" />
+    <xacro:property name="link_4_mesh_no" value="4" />
+    <xacro:property name="link_5_mesh_no" value="4" />
+    <xacro:property name="link_6_mesh_no" value="56" />
     <xacro:property name="joint_base" value="joint_base" />
     <xacro:property name="joint_base_type" value="fixed" />
@@ -67,4 +70,18 @@
     <xacro:property name="joint_4_lower_limit" value="${-2*J_PI}" />
     <xacro:property name="joint_4_upper_limit" value="${2*J_PI}" />
+    <xacro:property name="joint_5" value="joint_5" />
+    <xacro:property name="joint_5_type" value="continuous" />
+    <xacro:property name="joint_5_axis_xyz" value="0 0 1" />
+    <xacro:property name="joint_5_origin_xyz" value="0 -0.03703 -0.06414" />
+    <xacro:property name="joint_5_origin_rpy" value="${J_PI/3} 0 ${J_PI}" />
+    <xacro:property name="joint_5_lower_limit" value="${-2*J_PI}" />
+    <xacro:property name="joint_5_upper_limit" value="${2*J_PI}" />
+    <xacro:property name="joint_6" value="joint_6" />
+    <xacro:property name="joint_6_type" value="continuous" />
+    <xacro:property name="joint_6_axis_xyz" value="0 0 1" />
+    <xacro:property name="joint_6_origin_xyz" value="0 -0.03703 -0.06414" />
+    <xacro:property name="joint_6_origin_rpy" value="${J_PI/3} 0 ${J_PI}" />
+    <xacro:property name="joint_6_lower_limit" value="${-2*J_PI}" />
+    <xacro:property name="joint_6_upper_limit" value="${2*J_PI}" />
     <xacro:property name="joint_end_effector" value="end_effector_offset" />
     <xacro:property name="joint_end_effector_type" value="fixed" />
@@ -72,5 +89,5 @@
     <xacro:property name="joint_end_effector_origin_xyz" value="0 0 -0.1600" />
     <xacro:property name="joint_end_effector_origin_rpy" value="${J_PI} 0 ${J_PI/2}" />
-    <xacro:macro name="m1n4s200" params="base_parent prefix:=m1n4s200">
+    <xacro:macro name="m1n6s" params="base_parent prefix:=m1n6s200">
         <xacro:gazebo_config robot_namespace="${prefix}"/>
         <xacro:kinova_armlink link_name="${prefix}_link_base" link_mesh="${link_base_mesh}" mesh_no="${link_base_mesh_no}"/>
@@ -84,7 +101,10 @@
         <xacro:kinova_armlink link_name="${prefix}_link_4" link_mesh="${link_4_mesh}" use_ring_mesh="true" ring_mesh="ring_small" mesh_no="${link_4_mesh_no}"/>
         <xacro:kinova_armjoint joint_name="${prefix}_joint_4" type="${joint_4_type}" parent="${prefix}_link_3" child="${prefix}_link_4" joint_axis_xyz="${joint_4_axis_xyz}" joint_origin_xyz="${joint_4_origin_xyz}" joint_origin_rpy="${joint_4_origin_rpy}" joint_lower_limit="${joint_4_lower_limit}" joint_upper_limit="${joint_4_upper_limit}"/>
+        <xacro:kinova_armlink link_name="${prefix}_link_5" link_mesh="${link_5_mesh}" use_ring_mesh="true" ring_mesh="ring_small" mesh_no="${link_5_mesh_no}"/>
+        <xacro:kinova_armjoint joint_name="${prefix}_joint_5" type="${joint_5_type}" parent="${prefix}_link_4" child="${prefix}_link_5" joint_axis_xyz="${joint_5_axis_xyz}" joint_origin_xyz="${joint_5_origin_xyz}" joint_origin_rpy="${joint_5_origin_rpy}" joint_lower_limit="${joint_5_lower_limit}" joint_upper_limit="${joint_5_upper_limit}"/>
+        <xacro:kinova_armlink link_name="${prefix}_link_6" link_mesh="${link_6_mesh}" use_ring_mesh="true" ring_mesh="ring_small" mesh_no="${link_6_mesh_no}"/>
+        <xacro:kinova_armjoint joint_name="${prefix}_joint_6" type="${joint_6_type}" parent="${prefix}_link_5" child="${prefix}_link_6" joint_axis_xyz="${joint_6_axis_xyz}" joint_origin_xyz="${joint_6_origin_xyz}" joint_origin_rpy="${joint_6_origin_rpy}" joint_lower_limit="${joint_6_lower_limit}" joint_upper_limit="${joint_6_upper_limit}"/>
         <xacro:kinova_virtual_link link_name="${prefix}_end_effector"/>
-        <xacro:kinova_virtual_joint joint_name="joint_end_effector" type="${joint_end_effector_type}" parent="${prefix}_link_4" child="${prefix}_end_effector" joint_axis_xyz="${joint_end_effector_axis_xyz}" joint_origin_xyz="${joint_end_effector_origin_xyz}" joint_origin_rpy="${joint_end_effector_origin_rpy}" joint_lower_limit="0" joint_upper_limit="0"/>
-        <xacro:kinova_2fingers link_hand="${prefix}_link_4" prefix="${prefix}_"/>
+        <xacro:kinova_virtual_joint joint_name="${prefix}_joint_end_effector" type="${joint_end_effector_type}" parent="${prefix}_link_6" child="${prefix}_end_effector" joint_axis_xyz="${joint_end_effector_axis_xyz}" joint_origin_xyz="${joint_end_effector_origin_xyz}" joint_origin_rpy="${joint_end_effector_origin_rpy}" joint_lower_limit="0" joint_upper_limit="0"/>
     </xacro:macro>
 </root>

File: iter_moveit/m1n6s_robotiq85_moveit_config/urdf/m1n6s_robotiq85_standalone.xacro (robot description, xacro)
@@ -13,6 +13,5 @@
     xmlns:renderable="http://playerstage.sourceforge.net/gazebo/xmlschema/#renderable"
     xmlns:physics="http://playerstage.sourceforge.net/gazebo/xmlschema/#physics"
-	xmlns:xacro="http://ros.org/wiki/xacro" name="m1n6s200">
-  <xacro:include filename="$(find kinova_description)/urdf/m1n6s200.xacro"/>
+	xmlns:xacro="http://ros.org/wiki/xacro" name="m1n6s_robotiq85">
   <link name="root">
     <visual>
@@ -37,5 +36,18 @@
     <origin xyz="0 0 0" rpy="0 0 0" />
   </joint>
-  <xacro:property name="robot_root" value="root" />
-  <xacro:m1n6s200  base_parent="${robot_root}"/>
+	<!-- THE ROBOT -->
+	<link name="base_link"/>
+	<!-- M1N6S Mico Arm -->
+	<xacro:include filename="$(find m1n6s_robotiq85_moveit_config)/urdf/m1n6s.xacro" />
+  <joint name="base_joint" type="fixed">
+		<parent link="root" />
+		<child link = "base_link" />
+		<origin xyz="0.0 0.0 0.0" rpy="0.0 0.0 0.0" />
+	</joint>
+  <xacro:m1n6s base_parent="base_link" />
+	<!-- Robotiq 85-->
+	<xacro:include filename="$(find robotiq_85_description)/urdf/robotiq_85_gripper.urdf.xacro" />
+	<xacro:robotiq_85_gripper prefix="simple_gripper_" parent="m1n6s200_end_effector">
+	  <origin xyz="0 0 0" rpy="${pi/2} -${pi/2} 0" />
+	</xacro:robotiq_85_gripper>
 </robot>

Commit message: URDF robotiq working in sim

File: iter_moveit/m1n6s_robotiq85_moveit_config/urdf/m1n6s.xacro (robot description, xacro)
@@ -87,5 +87,5 @@
     <xacro:property name="joint_end_effector_type" value="fixed" />
     <xacro:property name="joint_end_effector_axis_xyz" value="0 0 0" />
-    <xacro:property name="joint_end_effector_origin_xyz" value="0 0 -0.1600" />
+    <xacro:property name="joint_end_effector_origin_xyz" value="0 0 -0.06" /> <!-- -0.1600 -->
     <xacro:property name="joint_end_effector_origin_rpy" value="${J_PI} 0 ${J_PI/2}" />
     <xacro:macro name="m1n6s" params="base_parent prefix:=m1n6s200">

Commit message: correcting end-effector offset for robotiq adapter

File: iter_moveit/m1n6s_robotiq85_moveit_config/urdf/m1n6s.xacro (robot description, xacro)
@@ -87,5 +87,5 @@
     <xacro:property name="joint_end_effector_type" value="fixed" />
     <xacro:property name="joint_end_effector_axis_xyz" value="0 0 0" />
-    <xacro:property name="joint_end_effector_origin_xyz" value="0 0 -0.06" /> <!-- -0.1600 -->
+    <xacro:property name="joint_end_effector_origin_xyz" value="0 0 -0.0625" />
     <xacro:property name="joint_end_effector_origin_rpy" value="${J_PI} 0 ${J_PI/2}" />
     <xacro:macro name="m1n6s" params="base_parent prefix:=m1n6s200">

Commit message: current status: gripper not controllable with moveit

File: iter_moveit/m1n6s_robotiq85_moveit_config/urdf/m1n6s.xacro (robot description, xacro)
@@ -23,5 +23,5 @@
     <xacro:property name="link_4_mesh" value="wrist" />
     <xacro:property name="link_5_mesh" value="wrist" />
-    <xacro:property name="link_6_mesh" value="hand_2finger" />
+    <xacro:property name="link_6_mesh" value="kinova_robotiq_coupler" />
     <!--Used for conditional arguments for setting inertial parameters
         base 0, shoulder 1, arm 2, forearm 3, wrist 4, arm_mico 5,
@@ -80,5 +80,5 @@
     <xacro:property name="joint_6_type" value="continuous" />
     <xacro:property name="joint_6_axis_xyz" value="0 0 1" />
-    <xacro:property name="joint_6_origin_xyz" value="0 -0.03703 -0.06414" />
+    <xacro:property name="joint_6_origin_xyz" value="0 -0.03703 -0.06414" /> <!--value="0 -0.03703 -0.06414" />-->
     <xacro:property name="joint_6_origin_rpy" value="${J_PI/3} 0 ${J_PI}" />
     <xacro:property name="joint_6_lower_limit" value="${-2*J_PI}" />
@@ -87,6 +87,34 @@
     <xacro:property name="joint_end_effector_type" value="fixed" />
     <xacro:property name="joint_end_effector_axis_xyz" value="0 0 0" />
-    <xacro:property name="joint_end_effector_origin_xyz" value="0 0 -0.0625" />
+    <xacro:property name="joint_end_effector_origin_xyz" value="0 0 -0.051" />
     <xacro:property name="joint_end_effector_origin_rpy" value="${J_PI} 0 ${J_PI/2}" />
+    <xacro:macro name="kinova_finger_fake" params="prefix finger_number hand finger_origin_xyz finger_origin_rpy">
+        <link name="${prefix}link_finger_${finger_number}"></link>
+        <joint name="${prefix}joint_finger_${finger_number}" type="revolute">
+            <parent link="${hand}"/>
+            <child link="${prefix}link_finger_${finger_number}"/>
+            <axis xyz="0 0 1"/>
+            <origin xyz="${finger_origin_xyz}" rpy="${finger_origin_rpy}"/>
+            <limit lower="0" upper="2" effort="2000" velocity="1"/>
+        </joint>
+        <transmission name="${prefix}joint_finger_${finger_number}_trans">
+					<type>transmission_interface/SimpleTransmission</type>
+					<joint name="${prefix}joint_finger_${finger_number}">
+					  <hardwareInterface>EffortJointInterface</hardwareInterface>
+					</joint>
+					<actuator name="${prefix}joint_finger_${finger_number}_actuator">
+					<hardwareInterface>EffortJointInterface</hardwareInterface>
+					<mechanicalReduction>1</mechanicalReduction>
+					</actuator>
+		    </transmission>
+        <link name="${prefix}link_finger_tip_${finger_number}"></link>
+        <joint name="${prefix}joint_finger_tip_${finger_number}" type="fixed">
+            <parent link="${prefix}link_finger_${finger_number}"/>
+            <child link="${prefix}link_finger_tip_${finger_number}"/>
+            <axis xyz="0 0 1"/>
+            <origin xyz="0.044 -0.003 0" rpy="0 0 0"/>
+            <limit lower="0" upper="2" effort="2000" velocity="1"/>
+        </joint>
+    </xacro:macro>
     <xacro:macro name="m1n6s" params="base_parent prefix:=m1n6s200">
         <xacro:gazebo_config robot_namespace="${prefix}"/>
@@ -103,8 +131,29 @@
         <xacro:kinova_armlink link_name="${prefix}_link_5" link_mesh="${link_5_mesh}" use_ring_mesh="true" ring_mesh="ring_small" mesh_no="${link_5_mesh_no}"/>
         <xacro:kinova_armjoint joint_name="${prefix}_joint_5" type="${joint_5_type}" parent="${prefix}_link_4" child="${prefix}_link_5" joint_axis_xyz="${joint_5_axis_xyz}" joint_origin_xyz="${joint_5_origin_xyz}" joint_origin_rpy="${joint_5_origin_rpy}" joint_lower_limit="${joint_5_lower_limit}" joint_upper_limit="${joint_5_upper_limit}"/>
-        <xacro:kinova_armlink link_name="${prefix}_link_6" link_mesh="${link_6_mesh}" use_ring_mesh="true" ring_mesh="ring_small" mesh_no="${link_6_mesh_no}"/>
+        <!--<xacro:kinova_armlink link_name="${prefix}_link_6" link_mesh="${link_6_mesh}" use_ring_mesh="true" ring_mesh="ring_small" mesh_no="${link_6_mesh_no}"/>-->
+        <link name="${prefix}_link_6">
+          <visual>
+            <geometry>
+              <mesh filename="package://m1n6s_robotiq85_moveit_config/meshes/${link_6_mesh}.dae" />
+            </geometry>
+            <material name="carbon_fiber">
+              <color rgba="0.792156862745098 0.819607843137255 0.933333333333333 1" />
+            </material>
+          </visual>
+          <collision>
+            <geometry>
+              <mesh filename="package://m1n6s_robotiq85_moveit_config/meshes/${link_6_mesh}.stl" />
+            </geometry>
+          </collision>
+          <xacro:kinova_inertial mesh_no="${link_6_mesh_no}"/>
+        </link>
         <xacro:kinova_armjoint joint_name="${prefix}_joint_6" type="${joint_6_type}" parent="${prefix}_link_5" child="${prefix}_link_6" joint_axis_xyz="${joint_6_axis_xyz}" joint_origin_xyz="${joint_6_origin_xyz}" joint_origin_rpy="${joint_6_origin_rpy}" joint_lower_limit="${joint_6_lower_limit}" joint_upper_limit="${joint_6_upper_limit}"/>
         <xacro:kinova_virtual_link link_name="${prefix}_end_effector"/>
         <xacro:kinova_virtual_joint joint_name="${prefix}_joint_end_effector" type="${joint_end_effector_type}" parent="${prefix}_link_6" child="${prefix}_end_effector" joint_axis_xyz="${joint_end_effector_axis_xyz}" joint_origin_xyz="${joint_end_effector_origin_xyz}" joint_origin_rpy="${joint_end_effector_origin_rpy}" joint_lower_limit="0" joint_upper_limit="0"/>
+        <!-- Need to enumerate fingers for hardware interface but will ignore them -->
+        <!-- finger1 Rot := Ry((1/2)*Pi) . Rx(Pi) . Rz(-52.8*((1/180)*Pi)) -->
+        <xacro:kinova_finger_fake prefix="${prefix}_" finger_number="1" hand="${prefix}_link_6" finger_origin_xyz="-0.0025 0.03095 -0.11482" finger_origin_rpy="-1.570796327 .649262481663582 1.57079632679490"/>
+        <!-- finger2 Rot := Ry((1/2)*Pi) . Rz(-52.8*((1/180)*Pi))  -->
+        <xacro:kinova_finger_fake prefix="${prefix}_" finger_number="2" hand="${prefix}_link_6" finger_origin_xyz="-0.0025 -0.03095 -0.11482" finger_origin_rpy="-1.570796327 .649262481663582 -1.57079632679490"/>
     </xacro:macro>
 </root>

Commit message: working on gripper control

File: iter_moveit/m1n6s_robotiq85_moveit_config/urdf/m1n6s.xacro (robot description, xacro)
@@ -88,5 +88,5 @@
     <xacro:property name="joint_end_effector_axis_xyz" value="0 0 0" />
     <xacro:property name="joint_end_effector_origin_xyz" value="0 0 -0.051" />
-    <xacro:property name="joint_end_effector_origin_rpy" value="${J_PI} 0 ${J_PI/2}" />
+    <xacro:property name="joint_end_effector_origin_rpy" value="${J_PI} 0 0" /> <!-- value="${J_PI} 0 ${J_PI/2}" -->
     <xacro:macro name="kinova_finger_fake" params="prefix finger_number hand finger_origin_xyz finger_origin_rpy">
         <link name="${prefix}link_finger_${finger_number}"></link>

File: iter_moveit/m1n6s_robotiq85_moveit_config/urdf/m1n6s_robotiq85.xacro (robot description, xacro)
@@ -1,4 +1,13 @@
 <?xml version="1.0"?>
 <robot name="m1n6s_robotiq85" xmlns:xacro="http://ros.org/wiki/xacro">
+	<link name="root">
+  </link>
+  <!-- for gazebo -->
+  <link name="world"/>
+  <joint name="connect_root_and_world" type="fixed">
+    <child link="root" />
+    <parent link="world" />
+    <origin xyz="0 0 0" rpy="0 0 0" />
+  </joint>
 	<!-- THE ROBOT -->
 	<link name="base_link" />
